File: simm-30-4mb.kicad_pcb (KiCad board)
At the start: 4 copper layers, 77.7 x 19 mm, 7 parts, among them J2 Conn_01x30, U1 511400, U2 511400

Commit message: Finished routing. Now need to do the board outline more
Parts:
- removed the C3 at (176.0, 76.2)
- removed the C3 at (159.5, 75.9)
- added C3: 100n, stdpads:C_1206, F.Cu at (137.7, 76.7)
- added C3: 100n, stdpads:C_1206, F.Cu at (159.3, 76.7)
- added C4: 100n, stdpads:C_1206, F.Cu at (176.5, 76.7)
- U1, U2: footprint stdpads:SOP-24-26-300mil -> stdpads:SOJ-24-26-300mil
- moved C1 0.77 mm to (103.5, 76.7)
- moved C2 0.77 mm to (125.1, 76.7)
- moved U1 0.13 mm to (148.6, 73.7)
- moved U2 0.13 mm to (114.3, 73.7)
Connections:
- J2 pad 11: /1A0 -> /1A6
- J2 pad 12: /1A6 -> /1A1
- J2 pad 14: /1A1 -> /1A7
- J2 pad 15: /1A5 -> /1A0
- J2 pad 17: /1A2 -> /1A8
- J2 pad 18: /1A4 -> /1A10
- J2 pad 19: /1A3 -> /1A9
- J2 pad 4: /1A9 -> /1A4
- J2 pad 5: /1A8 -> /1A3
- J2 pad 7: /1A10 -> /1A5
- J2 pad 8: /1A7 -> /1A2
- U1 pad 22: /~OE~ -> GND
- U2 pad 10: /1A0 -> /1A1
- U2 pad 11: /1A10 -> /1A0
- U2 pad 12: /1A9 -> /1A10
- U2 pad 15: /1A8 -> /1A9
- U2 pad 16: /1A7 -> /1A8
- U2 pad 17: /1A6 -> /1A7
- U2 pad 18: /1A5 -> /1A6
- U2 pad 19: /1A4 -> /1A5
- U2 pad 21: /1A3 -> /1A4
- U2 pad 22: /~OE~ -> GND
- U2 pad 8: /1A2 -> /1A3
- U2 pad 9: /1A1 -> /1A2
Routing:
- net /1A5: track 112.8 -> 57.8 mm
- net /1A4: track 114.1 -> 63.4 mm
- net /1A3: track 20.9 -> 63.2 mm
- net /1A2: track 21.5 -> 60.6 mm
- net /~WE~: track 20.0 -> 57.0 mm, vias 1 -> 2
- net /~CASP~: track 34.8 -> 0.00 mm
- net +5V: track 0.00 -> 29.6 mm, vias 0 -> 14
- net GND: track 0.00 -> 25.3 mm, vias 0 -> 42
- net /1A10: track 48.6 -> 72.6 mm
- net /1A8: track 45.5 -> 69.3 mm
- net /1A9: track 45.4 -> 66.9 mm
- net /1A7: track 50.0 -> 65.5 mm
- net /1A0: track 59.8 -> 68.4 mm
- net /~RAS~: track 76.7 -> 69.2 mm, vias 1 -> 2
- net /~CAS~: track 48.7 -> 55.6 mm, vias 2 -> 3
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- added copper zone on In2.Cu, net +5V
- added copper zone on B.Cu, net GND
- added copper zone on In1.Cu, net GND
Other:
- net class Default: clearance 0.127 -> 0.1524; trace_width 0.127 -> 0.1524
- rule trace_clearance: 0.127 -> 0.1524

Commit message: Submitted to JLCPCB
Parts:
- removed the C3 at (137.7, 76.7)
- removed the C3 at (159.3, 76.7)
- removed J2: Conn_01x30, stdpads:Memory_SIMM_30
- added C3: 100n, stdpads:C_0805, F.Cu at (119.4, 93.3)
- added C5: 100n, stdpads:C_0805, F.Cu at (157.5, 93.3)
- added J1: Conn_01x30, stdpads:SIMM-30_Edge, F.Cu at (120.7, 99.8)
- C1, C2, C4: footprint stdpads:C_1206 -> stdpads:C_0805
- U1, U2: value 511400 -> AS4C4M4; footprint stdpads:SOJ-24-26-300mil -> stdpads:SOP-24-26-300mil
- moved C4 40.4 mm to (139.7, 93.3)
- moved C2 25.8 mm to (105.4, 93.3)
- moved U1 24.9 mm to (129.5, 89.7)
- moved U2 24.9 mm to (95.2, 89.7)
- moved C1 24.8 mm to (85.1, 93.3)
Connections:
- U1 pad 6: Net-(U1-Pad6) -> (no net)
- U2 pad 6: Net-(U2-Pad6) -> (no net)
Routing:
- net GND: track 25.3 -> 22.3 mm, vias 42 -> 121
- net +5V: track 29.6 -> 26.8 mm, vias 14 -> 15
- net /~WE~: track 57.0 -> 57.6 mm
- added copper zone on B.Cu, net +5V
- added copper zone on In2.Cu, net GND
- removed copper zone on In2.Cu, net +5V
- removed copper zone on B.Cu, net GND
Other:
- board size 77.7 x 19 mm -> 88.9 x 19 mm
- rule solder_mask_min_width: 0.1524 -> 0.127
- board text added: "4 MB RAM"
- board text added: "4190A"
- board text added: "GW"
- board text added: "Garrett’s Workshop"
- board text added: "JLCJLCJLC"
