File: simm-30-4mb.kicad_pcb (KiCad board)
At the start: 4 copper layers, 88.9 x 19 mm, 8 parts, among them J1 Conn_01x30, U1 AS4C4M4, U2 AS4C4M4

Commit message: Extended edge connector pads downward
Parts:
- J1: value Conn_01x30 -> DRAM-SIMM-30
