File: simm-30-4mb.sch (KiCad schematic (older format))
At the start: 6 parts, among them J2 Conn_01x30, U1 511400, U2 511400

Commit message: Finished routing. Now need to do the board outline more
Parts:
- added C4: 100n, stdpads:C_1206, symbol Device:C_Small
Connections:
- net ~OE~ is gone; now on net GND: U1.22 (Pin_22), U2.22 (Pin_22)
- net +5V: now also C4.1
- net 1A0: now also J2.15 (Pin_15), U2.11 (Pin_11); no longer J2.11 (Pin_11), U2.10 (Pin_10)
- net 1A1: now also J2.12 (Pin_12), U2.10 (Pin_10); no longer J2.14 (Pin_14), U2.9 (Pin_9)
- net 1A10: now also J2.18 (Pin_18), U2.12 (Pin_12); no longer J2.7 (Pin_7), U2.11 (Pin_11)
- net 1A2: now also J2.8 (Pin_8), U2.9 (Pin_9); no longer J2.17 (Pin_17), U2.8 (Pin_8)
- net 1A3: now also J2.5 (Pin_5), U2.8 (Pin_8); no longer J2.19 (Pin_19), U2.21 (Pin_21)
- net 1A4: now also J2.4 (Pin_4), U2.21 (Pin_21); no longer J2.18 (Pin_18), U2.19 (Pin_19)
- net 1A5: now also J2.7 (Pin_7), U2.19 (Pin_19); no longer J2.15 (Pin_15), U2.18 (Pin_18)
- net 1A6: now also J2.11 (Pin_11), U2.18 (Pin_18); no longer J2.12 (Pin_12), U2.17 (Pin_17)
- net 1A7: now also J2.14 (Pin_14), U2.17 (Pin_17); no longer J2.8 (Pin_8), U2.16 (Pin_16)
- net 1A8: now also J2.17 (Pin_17), U2.16 (Pin_16); no longer J2.5 (Pin_5), U2.15 (Pin_15)
- net 1A9: now also J2.19 (Pin_19), U2.15 (Pin_15); no longer J2.4 (Pin_4), U2.12 (Pin_12)
- net GND: now also C4.2
Other:
- moved on the sheet: C1, C2, C3
Changed lines of the file:
@@
 NoConn ~ 5500 4700
 NoConn ~ 6000 4700
-$Comp
-L Device:C_Small C1
-U 1 1 5C2E290A
-P 2800 4200
-F 0 "C1" H 2892 4246 50  0000 L CNN
-F 1 "100n" H 2892 4155 50  0000 L CNN
-F 2 "stdpads:C_1206" H 2800 4200 50  0001 C CNN
-F 3 "~" H 2800 4200 50  0001 C CNN
-	1    2800 4200
-	1    0    0    -1
-$EndComp
-$Comp
-L Device:C_Small C2
-U 1 1 5C2E296A
-P 3200 4200
-F 0 "C2" H 3292 4246 50  0000 L CNN
-F 1 "100n" H 3292 4155 50  0000 L CNN
-F 2 "stdpads:C_1206" H 3200 4200 50  0001 C CNN
-F 3 "~" H 3200 4200 50  0001 C CNN
-	1    3200 4200
-	1    0    0    -1
-$EndComp
-Wire Wire Line
-	3200 4300 2800 4300
-$Comp
-L power:+5V #PWR0113
-U 1 1 5C2E299D
-P 2800 4100
-F 0 "#PWR0113" H 2800 3950 50  0001 C CNN
-F 1 "+5V" H 2800 4250 50  0000 C CNN
-F 2 "" H 2800 4100 50  0001 C CNN
-F 3 "" H 2800 4100 50  0001 C CNN
-	1    2800 4100
-	1    0    0    -1
-$EndComp
-Connection ~ 2800 4100
-Wire Wire Line
-	2800 4100 3200 4100
-$Comp
-L power:GND #PWR0114
-U 1 1 5C2E29CC
-P 3600 4300
-F 0 "#PWR0114" H 3600 4050 50  0001 C CNN
-F 1 "GND" H 3600 4150 50  0000 C CNN
-F 2 "" H 3600 4300 50  0001 C CNN
-F 3 "" H 3600 4300 50  0001 C CNN
-	1    3600 4300
-	1    0    0    -1
-$EndComp
 Text Label 6000 4600 0    50   ~ 0
 2A9
-Text Label 1950 5750 0    50   ~ 0
-1A10
-Text Label 1950 6950 0    50   ~ 0
-1A2
-Text Label 1950 6550 0    50   ~ 0
-1A1
-Text Label 1950 6150 0    50   ~ 0
-1A0
-Text Label 1950 7350 0    50   ~ 0
-1A3
-Text Label 1950 5650 0    50   ~ 0
-1A8
-Text Label 1950 6050 0    50   ~ 0
-1A7
-Text Label 1950 6450 0    50   ~ 0
-1A6
-Text Label 1950 6850 0    50   ~ 0
-1A5
-Text Label 1950 7250 0    50   ~ 0
-1A4
-Text Label 1950 5850 0    50   ~ 0
-2A2
-Text Label 1950 7050 0    50   ~ 0
-2A10
-Text Label 1950 6650 0    50   ~ 0
-2A0
-Text Label 1950 6250 0    50   ~ 0
-2A1
-Text Label 1950 7450 0    50   ~ 0
-2A9
-Text Label 1950 7150 0    50   ~ 0
-2A8
-Text Label 1950 6750 0    50   ~ 0
-2A7
-Text Label 1950 6350 0    50   ~ 0
-2A6
-Text Label 1950 5950 0    50   ~ 0
-2A5
-Text Label 1950 5550 0    50   ~ 0
-2A4
-Text Label 1750 6000 2    50   ~ 0
-A3
-Text Label 1750 5800 2    50   ~ 0
-A2
-Text Label 1750 5600 2    50   ~ 0
-A1
-Text Label 1750 5400 2    50   ~ 0
-A0
-Text Label 1750 7400 2    50   ~ 0
-A10
-Text Label 1750 7000 2    50   ~ 0
-A8
-Text Label 1750 6800 2    50   ~ 0
-A7
-Text Label 1750 6600 2    50   ~ 0
-A6
-Text Label 1750 6400 2    50   ~ 0
-A5
-Text Label 1750 6200 2    50   ~ 0
-A4
 Wire Wire Line
 	1850 7400 1850 7350
@@
 Text Label 6000 5200 0    50   ~ 0
 2A4
-Text Label 1750 7200 2    50   ~ 0
-A9
-Text Label 1950 5350 0    50   ~ 0
-2A3
-Text Label 1950 5450 0    50   ~ 0
-1A9
 Wire Wire Line
 	1850 7200 1850 7150
@@
 	1750 7200 1850 7200
 $Comp
+L Device:C_Small C1
+U 1 1 5C2E290A
+P 2400 4200
+F 0 "C1" H 2492 4246 50  0000 L CNN
+F 1 "100n" H 2492 4155 50  0000 L CNN
+F 2 "stdpads:C_1206" H 2400 4200 50  0001 C CNN
+F 3 "~" H 2400 4200 50  0001 C CNN
+	1    2400 4200
+	1    0    0    -1
+$EndComp
+$Comp
+L Device:C_Small C2
+U 1 1 5C2E296A
+P 2800 4200
+F 0 "C2" H 2892 4246 50  0000 L CNN
+F 1 "100n" H 2892 4155 50  0000 L CNN
+F 2 "stdpads:C_1206" H 2800 4200 50  0001 C CNN
+F 3 "~" H 2800 4200 50  0001 C CNN
+	1    2800 4200
+	1    0    0    -1
+$EndComp
+Wire Wire Line
+	2800 4300 2400 4300
+$Comp
+L power:+5V #PWR0113
+U 1 1 5C2E299D
+P 2400 4100
+F 0 "#PWR0113" H 2400 3950 50  0001 C CNN
+F 1 "+5V" H 2400 4250 50  0000 C CNN
+F 2 "" H 2400 4100 50  0001 C CNN
+F 3 "" H 2400 4100 50  0001 C CNN
+	1    2400 4100
+	1    0    0    -1
+$EndComp
+Connection ~ 2400 4100
+Wire Wire Line
+	2400 4100 2800 4100
+$Comp
 L Device:C_Small C3
 U 1 1 5C2EDC35
+P 3200 4200
+F 0 "C3" H 3292 4246 50  0000 L CNN
+F 1 "100n" H 3292 4155 50  0000 L CNN
+F 2 "stdpads:C_1206" H 3200 4200 50  0001 C CNN
+F 3 "~" H 3200 4200 50  0001 C CNN
+	1    3200 4200
+	1    0    0    -1
+$EndComp
+Wire Wire Line
+	3200 4100 2800 4100
+Connection ~ 2800 4100
+Wire Wire Line
+	2800 4300 3200 4300
+Connection ~ 2800 4300
+Connection ~ 3200 4300
+$Comp
+L power:GND #PWR0114
+U 1 1 5C2E29CC
+P 3600 4300
+F 0 "#PWR0114" H 3600 4050 50  0001 C CNN
+F 1 "GND" H 3600 4150 50  0000 C CNN
+F 2 "" H 3600 4300 50  0001 C CNN
+F 3 "" H 3600 4300 50  0001 C CNN
+	1    3600 4300
+	1    0    0    -1
+$EndComp
+Wire Wire Line
+	3200 4300 3600 4300
+Connection ~ 3600 4300
+Wire Wire Line
+	3600 4100 3200 4100
+Connection ~ 3200 4100
+$Comp
+L Device:C_Small C4
+U 1 1 5D1301A9
 P 3600 4200
-F 0 "C3" H 3692 4246 50  0000 L CNN
+F 0 "C4" H 3692 4246 50  0000 L CNN
 F 1 "100n" H 3692 4155 50  0000 L CNN
 F 2 "stdpads:C_1206" H 3600 4200 50  0001 C CNN
@@
 	1    0    0    -1
 $EndComp
-Wire Wire Line
-	3600 4100 3200 4100
-Connection ~ 3200 4100
-Wire Wire Line
-	3200 4300 3600 4300
-Connection ~ 3200 4300
-Connection ~ 3600 4300
+$Comp
+L power:GND #PWR0115
+U 1 1 5D14DFC9
+P 6200 4500
+F 0 "#PWR0115" H 6200 4250 50  0001 C CNN
+F 1 "GND" H 6200 4350 50  0000 C CNN
+F 2 "" H 6200 4500 50  0001 C CNN
+F 3 "" H 6200 4500 50  0001 C CNN
+	1    6200 4500
+	1    0    0    -1
+$EndComp
+Wire Wire Line
+	6200 4500 6000 4500
+$Comp
+L power:GND #PWR0116
+U 1 1 5D14FA7D
+P 4800 4500
+F 0 "#PWR0116" H 4800 4250 50  0001 C CNN
+F 1 "GND" H 4800 4350 50  0000 C CNN
+F 2 "" H 4800 4500 50  0001 C CNN
+F 3 "" H 4800 4500 50  0001 C CNN
+	1    4800 4500
+	1    0    0    -1
+$EndComp
+Wire Wire Line
+	4800 4500 4600 4500
+Text Label 1950 5650 0    50   ~ 0
+2A10
+Text Label 1950 5450 0    50   ~ 0
+2A9
+Text Label 1950 5850 0    50   ~ 0
+2A8
+Text Label 1950 6050 0    50   ~ 0
+2A0
+Text Label 1950 6250 0    50   ~ 0
+2A7
+Text Label 1950 6450 0    50   ~ 0
+2A1
+Text Label 1950 6850 0    50   ~ 0
+2A2
+Text Label 1950 7050 0    50   ~ 0
+2A5
+Text Label 1950 6650 0    50   ~ 0
+2A6
+Text Label 1950 7250 0    50   ~ 0
+2A3
+Text Label 1950 7450 0    50   ~ 0
+2A4
+Text Label 1750 6000 2    50   ~ 0
+A3
+Text Label 1750 5800 2    50   ~ 0
+A2
+Text Label 1750 5600 2    50   ~ 0
+A1
+Text Label 1750 5400 2    50   ~ 0
+A0
+Text Label 1750 7000 2    50   ~ 0
+A8
+Text Label 1750 6800 2    50   ~ 0
+A7
+Text Label 1750 6600 2    50   ~ 0
+A6
+Text Label 1750 6400 2    50   ~ 0
+A5
+Text Label 1750 6200 2    50   ~ 0
+A4
+Text Label 1750 7200 2    50   ~ 0
+A9
+Text Label 1750 7400 2    50   ~ 0
+A10
+Text Label 1950 5350 0    50   ~ 0
+1A4
+Text Label 1950 5550 0    50   ~ 0
+1A3
+Text Label 1950 5750 0    50   ~ 0
+1A5
+Text Label 1950 5950 0    50   ~ 0
+1A2
+Text Label 1950 6150 0    50   ~ 0
+1A6
+Text Label 1950 6350 0    50   ~ 0
+1A1
+Text Label 1950 6550 0    50   ~ 0
+1A7
+Text Label 1950 6750 0    50   ~ 0
+1A0
+Text Label 1950 6950 0    50   ~ 0
+1A8
+Text Label 1950 7150 0    50   ~ 0
+1A10
+Text Label 1950 7350 0    50   ~ 0
+1A9
 $EndSCHEMATC

Commit message: Submitted to JLCPCB
Parts:
- removed U1, U2: 511400, stdpads:SOJ-24-26-300mil, symbol Connector_Generic:Conn_02x13_Counter_Clockwise
- added C5: 100n, stdpads:C_0805, symbol Device:C_Small
- added U1, U2: AS4C4M4, stdpads:SOP-24-26-300mil, symbol stdparts:AS4C4M4
- C1, C2, C3, C4: footprint stdpads:C_1206 -> stdpads:C_0805
- J1: renamed from J2; footprint stdpads:Memory_SIMM_30 -> stdpads:SIMM-30_Edge
Connections:
- net +5V: now also C5.1, U1.1 (VDD), U1.13 (VDD), U2.1 (VDD), U2.13 (VDD)
- net 1A0: now also U1.9 (A0), U2.11 (A2)
- net 1A1: now also U1.10 (A1), U2.10 (A1)
- net 1A10: now also U1.8 (A10), U2.12 (A3)
- net 1A2: now also U1.11 (A2), U2.9 (A0)
- net 1A3: now also U1.12 (A3), U2.8 (A10)
- net 1A4: now also U1.15 (A4), U2.21 (A9)
- net 1A5: now also U1.16 (A5), U2.19 (A8)
- net 1A6: now also U1.17 (A6), U2.18 (A7)
- net 1A7: now also U1.18 (A7), U2.17 (A6)
- net 1A8: now also U1.19 (A8), U2.16 (A5)
- net 1A9: now also U1.21 (A9), U2.15 (A4)
- net D0: now also U2.25 (I/O3)
- net D1: now also U2.2 (I/O0)
- net D2: now also U2.24 (I/O2)
- net D3: now also U2.3 (I/O1)
- net D4: now also U1.25 (I/O3)
- net D5: now also U1.2 (I/O0)
- net D6: now also U1.24 (I/O2)
- net D7: now also U1.3 (I/O1)
- net GND: now also C5.2, U1.14 (GND), U1.22 (~OE~), U1.26 (GND), U2.14 (GND), U2.22 (~OE~), U2.26 (GND)
- net ~CAS~: now also U1.23 (~CAS~), U2.23 (~CAS~)
- net ~RAS~: now also U1.5 (~RAS~), U2.5 (~RAS~)
- net ~WE~: now also U1.4 (~WE~), U2.4 (~WE~)
- new net: U1.20 (NC), U1.7 (NC)
- new net: U2.20 (NC), U2.7 (NC)
- no-connect marks 6 -> 0

Commit message: Extended edge connector pads downward
Parts:
- J1: value Conn_01x30 -> DRAM-SIMM-30
- U1, U2: symbol stdparts:AS4C4M4 -> GW_RAM:DRAM-4Mx4-SOP-24
Other:
- moved on the sheet: U1, U2
Changed lines of the file:
@@
 EESchema Schematic File Version 4
-LIBS:simm-30-4mb-cache
-EELAYER 29 0
+EELAYER 30 0
 EELAYER END
 $Descr USLetter 11000 8500
@@
 P 4450 3450
 F 0 "J1" V 4574 3396 50  0000 C CNN
-F 1 "Conn_01x30" V 4665 3396 50  0000 C CNN
+F 1 "DRAM-SIMM-30" V 4665 3396 50  0000 C CNN
 F 2 "stdpads:SIMM-30_Edge" H 4450 3450 50  0001 C CNN
 F 3 "~" H 4450 3450 50  0001 C CNN
@@
 Text Label 5850 3250 1    50   ~ 0
 DP
-Text Label 4200 7000 0    50   ~ 0
+Text Label 4200 7050 0    50   ~ 0
 ~OE~
+Text Label 3400 6950 2    50   ~ 0
+1A8
 Text Label 3400 6850 2    50   ~ 0
-1A8
+1A7
 Text Label 3400 6750 2    50   ~ 0
-1A7
+1A6
 Text Label 3400 6650 2    50   ~ 0
-1A6
+1A5
 Text Label 3400 6550 2    50   ~ 0
-1A5
+1A4
 Text Label 3400 6450 2    50   ~ 0
-1A4
+1A3
 Text Label 3400 6350 2    50   ~ 0
-1A3
+1A2
 Text Label 3400 6250 2    50   ~ 0
-1A2
+1A1
 Text Label 3400 6150 2    50   ~ 0
-1A1
-Text Label 3400 6050 2    50   ~ 0
 1A0
-Text Label 3400 7050 2    50   ~ 0
+Text Label 3400 7150 2    50   ~ 0
 1A10
 Wire Wire Line
@@
 L power:GND #PWR0116
 U 1 1 5D14FA7D
-P 4400 7000
-F 0 "#PWR0116" H 4400 6750 50  0001 C CNN
-F 1 "GND" H 4400 6850 50  0000 C CNN
-F 2 "" H 4400 7000 50  0001 C CNN
-F 3 "" H 4400 7000 50  0001 C CNN
-	1    4400 7000
-	1    0    0    -1
-$EndComp
-Wire Wire Line
-	4400 7000 4200 7000
+P 4400 7050
+F 0 "#PWR0116" H 4400 6800 50  0001 C CNN
+F 1 "GND" H 4400 6900 50  0000 C CNN
+F 2 "" H 4400 7050 50  0001 C CNN
+F 3 "" H 4400 7050 50  0001 C CNN
+	1    4400 7050
+	1    0    0    -1
+$EndComp
+Wire Wire Line
+	4400 7050 4200 7050
 Text Label 1950 5650 0    50   ~ 0
 2A10
@@
 1A9
 $Comp
-L stdparts:AS4C4M4 U1
+L GW_RAM:DRAM-4Mx4-SOP-24 U1
 U 1 1 5D38F422
 P 3800 6650
-F 0 "U1" H 3800 7515 50  0000 C CNN
-F 1 "AS4C4M4" H 3800 7424 50  0000 C CNN
+F 0 "U1" H 3800 7300 50  0000 C CNN
+F 1 "AS4C4M4" H 3800 6000 50  0000 C CNN
 F 2 "stdpads:SOP-24-26-300mil" H 3800 5950 50  0001 C CNN
 F 3 "https://www.alliancememory.com/wp-content/uploads/pdf/AS6C8008.pdf" H 3800 6150 50  0001 C CNN
@@
 	1    0    0    -1
 $EndComp
-Text Label 3400 6950 2    50   ~ 0
+Text Label 3400 7050 2    50   ~ 0
 1A9
 $Comp
 L power:GND #PWR0105
 U 1 1 5D395DE3
-P 4200 7200
-F 0 "#PWR0105" H 4200 6950 50  0001 C CNN
-F 1 "GND" H 4200 7050 50  0000 C CNN
-F 2 "" H 4200 7200 50  0001 C CNN
-F 3 "" H 4200 7200 50  0001 C CNN
-	1    4200 7200
-	1    0    0    -1
-$EndComp
-Text Label 4200 6700 0    50   ~ 0
+P 4200 7150
+F 0 "#PWR0105" H 4200 6900 50  0001 C CNN
+F 1 "GND" H 4200 7000 50  0000 C CNN
+F 2 "" H 4200 7150 50  0001 C CNN
+F 3 "" H 4200 7150 50  0001 C CNN
+	1    4200 7150
+	1    0    0    -1
+$EndComp
+Text Label 4200 6750 0    50   ~ 0
 ~CAS~
-Text Label 4200 6800 0    50   ~ 0
+Text Label 4200 6850 0    50   ~ 0
 ~RAS~
-Text Label 4200 6900 0    50   ~ 0
+Text Label 4200 6950 0    50   ~ 0
 ~WE~
 Text Label 4200 6250 0    50   ~ 0
@@
 L power:+5V #PWR0106
 U 1 1 5D396692
-P 4200 6050
-F 0 "#PWR0106" H 4200 5900 50  0001 C CNN
-F 1 "+5V" H 4200 6200 50  0000 C CNN
-F 2 "" H 4200 6050 50  0001 C CNN
-F 3 "" H 4200 6050 50  0001 C CNN
-	1    4200 6050
-	1    0    0    -1
-$EndComp
-Text Label 5800 7050 0    50   ~ 0
+P 4200 6150
+F 0 "#PWR0106" H 4200 6000 50  0001 C CNN
+F 1 "+5V" H 4200 6300 50  0000 C CNN
+F 2 "" H 4200 6150 50  0001 C CNN
+F 3 "" H 4200 6150 50  0001 C CNN
+	1    4200 6150
+	1    0    0    -1
+$EndComp
+Text Label 5800 7100 0    50   ~ 0
 ~OE~
+Text Label 5000 7000 2    50   ~ 0
+2A8
 Text Label 5000 6900 2    50   ~ 0
-2A8
+2A7
 Text Label 5000 6800 2    50   ~ 0
-2A7
+2A6
 Text Label 5000 6700 2    50   ~ 0
-2A6
+2A5
 Text Label 5000 6600 2    50   ~ 0
-2A5
+2A4
 Text Label 5000 6500 2    50   ~ 0
-2A4
+2A3
 Text Label 5000 6400 2    50   ~ 0
-2A3
+2A2
 Text Label 5000 6300 2    50   ~ 0
-2A2
+2A1
 Text Label 5000 6200 2    50   ~ 0
-2A1
-Text Label 5000 6100 2    50   ~ 0
 2A0
-Text Label 5000 7100 2    50   ~ 0
+Text Label 5000 7200 2    50   ~ 0
 2A10
 $Comp
 L power:GND #PWR0107
 U 1 1 5D3999CF
-P 6000 7050
-F 0 "#PWR0107" H 6000 6800 50  0001 C CNN
-F 1 "GND" H 6000 6900 50  0000 C CNN
-F 2 "" H 6000 7050 50  0001 C CNN
-F 3 "" H 6000 7050 50  0001 C CNN
-	1    6000 7050
-	1    0    0    -1
-$EndComp
-Wire Wire Line
-	6000 7050 5800 7050
-$Comp
-L stdparts:AS4C4M4 U2
+P 6000 7100
+F 0 "#PWR0107" H 6000 6850 50  0001 C CNN
+F 1 "GND" H 6000 6950 50  0000 C CNN
+F 2 "" H 6000 7100 50  0001 C CNN
+F 3 "" H 6000 7100 50  0001 C CNN
+	1    6000 7100
+	1    0    0    -1
+$EndComp
+Wire Wire Line
+	6000 7100 5800 7100
+$Comp
+L GW_RAM:DRAM-4Mx4-SOP-24 U2
 U 1 1 5D3999D6
 P 5400 6700
-F 0 "U2" H 5400 7565 50  0000 C CNN
-F 1 "AS4C4M4" H 5400 7474 50  0000 C CNN
+F 0 "U2" H 5400 7350 50  0000 C CNN
+F 1 "AS4C4M4" H 5400 6050 50  0000 C CNN
 F 2 "stdpads:SOP-24-26-300mil" H 5400 6000 50  0001 C CNN
 F 3 "https://www.alliancememory.com/wp-content/uploads/pdf/AS6C8008.pdf" H 5400 6200 50  0001 C CNN
@@
 	1    0    0    -1
 $EndComp
-Text Label 5000 7000 2    50   ~ 0
+Text Label 5000 7100 2    50   ~ 0
 2A9
 $Comp
 L power:GND #PWR0108
 U 1 1 5D3999DD
-P 5800 7250
-F 0 "#PWR0108" H 5800 7000 50  0001 C CNN
-F 1 "GND" H 5800 7100 50  0000 C CNN
-F 2 "" H 5800 7250 50  0001 C CNN
-F 3 "" H 5800 7250 50  0001 C CNN
-	1    5800 7250
-	1    0    0    -1
-$EndComp
-Text Label 5800 6750 0    50   ~ 0
+P 5800 7200
+F 0 "#PWR0108" H 5800 6950 50  0001 C CNN
+F 1 "GND" H 5800 7050 50  0000 C CNN
+F 2 "" H 5800 7200 50  0001 C CNN
+F 3 "" H 5800 7200 50  0001 C CNN
+	1    5800 7200
+	1    0    0    -1
+$EndComp
+Text Label 5800 6800 0    50   ~ 0
 ~CAS~
-Text Label 5800 6850 0    50   ~ 0
+Text Label 5800 6900 0    50   ~ 0
 ~RAS~
-Text Label 5800 6950 0    50   ~ 0
+Text Label 5800 7000 0    50   ~ 0
 ~WE~
 $Comp
 L power:+5V #PWR0109
 U 1 1 5D3999EA
-P 5800 6100
-F 0 "#PWR0109" H 5800 5950 50  0001 C CNN
-F 1 "+5V" H 5800 6250 50  0000 C CNN
-F 2 "" H 5800 6100 50  0001 C CNN
-F 3 "" H 5800 6100 50  0001 C CNN
-	1    5800 6100
-	1    0    0    -1
-$EndComp
+P 5800 6200
+F 0 "#PWR0109" H 5800 6050 50  0001 C CNN
+F 1 "+5V" H 5800 6350 50  0000 C CNN
+F 2 "" H 5800 6200 50  0001 C CNN
+F 3 "" H 5800 6200 50  0001 C CNN
+	1    5800 6200
+	1    0    0    -1
+$EndComp
