File: 16MB-2chip-SOP/simm-30-16mb.kicad_pcb (KiCad board)
At the start: 4 copper layers, 88.9 x 20.8 mm, 14 parts, among them J1 DRAM-SIMM-30, U1 KM44C16104, U2 KM44C16104

Commit message: Some more tweaks
Routing:
- net GND: vias 70 -> 71
Changed lines of the file:
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@@
     (thickness 1.6)
     (drawings 16)
-    (tracks 427)
+    (tracks 428)
     (zones 0)
     (modules 14)
@@
   (via (at 123.825 82.55) (size 0.508) (drill 0.2) (layers F.Cu B.Cu) (net 9))
   (via (at 104.7115 91.3765) (size 0.508) (drill 0.2) (layers F.Cu B.Cu) (net 9))
-  (via (at 103.4415 91.2495) (size 0.508) (drill 0.2) (layers F.Cu B.Cu) (net 9))
+  (via (at 103.505 91.186) (size 0.508) (drill 0.2) (layers F.Cu B.Cu) (net 9))
   (via (at 102.362 90.932) (size 0.508) (drill 0.2) (layers F.Cu B.Cu) (net 9))
   (via (at 101.4095 90.4875) (size 0.508) (drill 0.2) (layers F.Cu B.Cu) (net 9))
@@
   (via (at 140.97 98.298) (size 0.508) (drill 0.2) (layers F.Cu B.Cu) (net 9))
   (via (at 130.81 98.3615) (size 0.508) (drill 0.2) (layers F.Cu B.Cu) (net 9))
+  (via (at 104.648 92.9005) (size 0.508) (drill 0.2) (layers F.Cu B.Cu) (net 9))
   (segment (start 121.92 96.058) (end 121.92 98.806) (width 0.1524) (layer F.Cu) (net 10))
   (segment (start 129.794 97.8535) (end 131.1275 97.8535) (width 0.1524) (layer F.Cu) (net 11))
@@
   (segment (start 100.33 87.9475) (end 101.0285 88.646) (width 0.1524) (layer F.Cu) (net 27))
   (segment (start 100.33 87.4395) (end 100.33 87.9475) (width 0.1524) (layer F.Cu) (net 27))
+  (segment (start 102.4255 89.3445) (end 104.14 91.059) (width 0.1524) (layer In2.Cu) (net 27))
+  (segment (start 104.14 94.8055) (end 108.1405 98.806) (width 0.1524) (layer In2.Cu) (net 27))
+  (segment (start 101.727 89.3445) (end 102.4255 89.3445) (width 0.1524) (layer In2.Cu) (net 27))
+  (segment (start 104.14 91.059) (end 104.14 94.8055) (width 0.1524) (layer In2.Cu) (net 27))
   (segment (start 108.1405 98.806) (end 109.22 98.806) (width 0.1524) (layer In2.Cu) (net 27))
-  (segment (start 104.14 94.8055) (end 108.1405 98.806) (width 0.1524) (layer In2.Cu) (net 27))
-  (segment (start 104.14 91.059) (end 104.14 94.8055) (width 0.1524) (layer In2.Cu) (net 27))
-  (segment (start 102.4255 89.3445) (end 104.14 91.059) (width 0.1524) (layer In2.Cu) (net 27))
-  (segment (start 101.727 89.3445) (end 102.4255 89.3445) (width 0.1524) (layer In2.Cu) (net 27))
   (segment (start 100.33 87.9475) (end 101.727 89.3445) (width 0.1524) (layer In2.Cu) (net 27))
   (segment (start 100.33 87.4395) (end 100.33 87.9475) (width 0.1524) (layer In2.Cu) (net 27))
   (via (at 97.79 87.4395) (size 0.508) (drill 0.2) (layers F.Cu B.Cu) (net 30))
-  (segment (start 97.79 88.2015) (end 101.6 92.0115) (width 0.1524) (layer In2.Cu) (net 30))
-  (segment (start 97.79 87.4395) (end 97.79 88.2015) (width 0.1524) (layer In2.Cu) (net 30))
   (segment (start 97.79 84.028) (end 97.79 87.4395) (width 0.1524) (layer F.Cu) (net 30))
   (segment (start 136.9695 89.281) (end 98.8695 89.281) (width 0.1524) (layer F.Cu) (net 30))
@@
   (segment (start 97.79 88.2015) (end 97.79 87.4395) (width 0.1524) (layer F.Cu) (net 30))
   (segment (start 138.43 84.028) (end 138.43 87.8205) (width 0.1524) (layer F.Cu) (net 30))
+  (segment (start 97.79 88.2015) (end 101.6 92.0115) (width 0.1524) (layer In2.Cu) (net 30))
   (segment (start 101.6 98.806) (end 101.6 92.0115) (width 0.1524) (layer In2.Cu) (net 30))
+  (segment (start 97.79 87.4395) (end 97.79 88.2015) (width 0.1524) (layer In2.Cu) (net 30))
   (segment (start 81.727 84.455) (end 81.727 86.487) (width 0.1524) (layer F.Cu) (net 33))
   (segment (start 81.727 84.455) (end 81.727 83.0605) (width 0.1524) (layer F.Cu) (net 33))
