File: GW4192-16MB-SOP/GW4192-SOP.kicad_pcb (KiCad board)
At the start: 4 copper layers, 88.9 x 20.8 mm, 14 parts, among them J1 DRAM-SIMM-30, U1 KM44C16104, U2 KM44C16104

Commit message: Fabbed
Routing:
- net +5V: track 31.3 -> 34.0 mm
Changed lines of the file:
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@@
     (thickness 1.6)
     (drawings 17)
-    (tracks 428)
+    (tracks 429)
     (zones 0)
     (modules 14)
@@
   )
   (setup
-    (last_trace_width 0.1524)
+    (last_trace_width 0.8)
     (user_trace_width 0.1524)
     (user_trace_width 0.254)
@@
   (segment (start 105.41 96.058) (end 105.41 94.615) (width 0.6) (layer F.Cu) (net 1))
   (via (at 105.41 94.615) (size 0.6) (drill 0.3) (layers F.Cu B.Cu) (net 1))
+  (segment (start 157.48 96.0755) (end 157.48 98.806) (width 0.8) (layer F.Cu) (net 1))
   (segment (start 88.9 100.076) (end 88.9 98.806) (width 0.1524) (layer F.Cu) (net 2))
   (segment (start 87.63 97.536) (end 88.9 98.806) (width 0.1524) (layer F.Cu) (net 2))
